File: 0017_RFID_Module_CR95HF.kicad_sch (KiCad schematic)
At the start: 32 parts, among them IC1 CR95HF-VMD5T, J1 Conn_01x03_Pin, J2 Conn_01x03_Pin, Y1 27.12Mhz

Commit message: Add files via upload
Parts:
- added D1: LED, LED_SMD:LED_0603_1608Metric, symbol Device:LED
- added R12: R, Resistor_SMD:R_0603_1608Metric, symbol Device:R
- added U1: ~, Moduler_:pin_header_5-3, symbol moduler_pin:air
- C1, C10, C11, C12, C13, C14, C15, C2, C3, C4, C5, C6, C7, C8, C9: footprint (none) -> Capacitor_SMD:C_0603_1608Metric
- FB1: footprint (none) -> Inductor_SMD:L_0603_1608Metric
- IC1: footprint QFN50P500X500X100-33N-D -> CR95HF:QFN50P500X500X100-33N-D
- J1, J2: footprint (none) -> Jumper:SolderJumper-3_P1.3mm_Open_Pad1.0x1.5mm
- R1, R10, R11, R2, R3, R4, R5, R6, R7, R8, R9: footprint (none) -> Resistor_SMD:R_0603_1608Metric
- Y1: footprint (none) -> Crystal:Crystal_SMD_5032-2Pin_5.0x3.2mm
Connections:
- net +3V3: now also R12.1, U1.8
- net CS: now also U1.3
- net GND: now also IC1.33 (THERMAL_PAD), D1.1 (K), U1.9
- net MISO: now also U1.2
- net MOSI: now also U1.1
- net RX: now also U1.11
- net SCK: now also U1.4
- net SSI_0: now also U1.12
- net SSI_1: now also U1.13
- net TX: now also U1.10
- new net: D1.2 (A), R12.2
- no-connect marks 0 -> 8
Other:
- moved on the sheet: AE1, C1, C10, C11, C12, C13, C14, C15, C2, C3, C4, C5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
